Commit message: python gui

File: src/omni_bot_description/urdf/omni_bot.urdf.xacro (robot description, xacro)
@@ -1,9 +1,16 @@
 <?xml version="1.0"?>
 <robot name="omni_bot" xmlns:xacro="http://www.ros.org/wiki/xacro">
-  <xacro:property name="base_radius" value="0.15"/>
-  <xacro:property name="base_height" value="0.08"/>
-  <xacro:property name="wheel_radius" value="0.04"/>
-  <xacro:property name="wheel_width" value="0.03"/>
+  <xacro:property name="base_radius" value="0.135"/>
+  <xacro:property name="base_height" value="0.235"/>
+  <xacro:property name="ground_clearance" value="0.02"/>
+  <xacro:property name="wheel_radius" value="0.05"/>
+  <xacro:property name="wheel_width" value="0.04"/>
   <xacro:property name="wheel_offset" value="0.16"/>
+  <link name="base_footprint"/>
+  <joint name="base_joint" type="fixed">
+    <parent link="base_footprint"/>
+    <child link="base_link"/>
+    <origin xyz="0 0 ${ground_clearance + base_height/2}" rpy="0 0 0"/>
+  </joint>
   <link name="base_link">
     <visual>
@@ -22,10 +29,10 @@
     <link name="${prefix}_wheel">
       <visual>
-        <origin rpy="1.5708 0 0"/>
+        <origin rpy="0 1.5708 0"/>
         <geometry><cylinder radius="${wheel_radius}" length="${wheel_width}"/></geometry>
         <material name="black"><color rgba="0.1 0.1 0.1 1"/></material>
       </visual>
       <collision>
-        <origin rpy="1.5708 0 0"/>
+        <origin rpy="0 1.5708 0"/>
         <geometry><cylinder radius="${wheel_radius}" length="${wheel_width}"/></geometry>
       </collision>
@@ -38,7 +45,9 @@
       <parent link="base_link"/>
       <child link="${prefix}_wheel"/>
-      <origin xyz="${wheel_offset * cos(angle_deg * pi / 180)} ${wheel_offset * sin(angle_deg * pi / 180)} 0"
+      <origin xyz="${wheel_offset * cos(angle_deg * pi / 180)}
+                   ${wheel_offset * sin(angle_deg * pi / 180)}
+                   ${wheel_radius - (ground_clearance + base_height/2)}"
               rpy="0 0 ${angle_deg * pi / 180}"/>
-      <axis xyz="0 1 0"/>
+      <axis xyz="1 0 0"/>
     </joint>
   </xacro:macro>

Commit message: v2

File: src/omni_bot_description/urdf/omni_bot.urdf.xacro (robot description, xacro)
@@ -4,4 +4,7 @@
   <xacro:property name="base_height" value="0.235"/>
   <xacro:property name="ground_clearance" value="0.02"/>
+  <!-- Heading marker ("face") dimensions -->
+  <xacro:property name="face_length" value="0.10"/>
+  <xacro:property name="face_width" value="0.03"/>
   <xacro:property name="wheel_radius" value="0.05"/>
   <xacro:property name="wheel_width" value="0.04"/>
@@ -26,4 +29,26 @@
     </inertial>
   </link>
+  <!-- Heading marker ("face"): yellow stick poking out of the robot's +x (front) side.
+       Visual only, no collision, so it never affects motion. -->
+  <link name="face_link">
+    <visual>
+      <geometry><box size="${face_length} ${face_width} ${face_width}"/></geometry>
+      <material name="yellow"><color rgba="1 0.8 0 1"/></material>
+    </visual>
+    <inertial>
+      <mass value="0.01"/>
+      <inertia ixx="0.000001" ixy="0" ixz="0" iyy="0.000001" iyz="0" izz="0.000001"/>
+    </inertial>
+  </link>
+  <joint name="face_joint" type="fixed">
+    <parent link="base_link"/>
+    <child link="face_link"/>
+    <!-- centre it so ~0.09 m sticks out past the base edge (0.01 m overlaps into the body) -->
+    <origin xyz="${base_radius + face_length/2 - 0.01} 0 0" rpy="0 0 0"/>
+  </joint>
+  <!-- Gazebo Classic often ignores URDF colours, so set it explicitly -->
+  <gazebo reference="face_link">
+    <material>Gazebo/Yellow</material>
+  </gazebo>
   <xacro:macro name="omni_wheel" params="prefix angle_deg">
     <link name="${prefix}_wheel">
